File: hardware/AirQualityMonitor/AirQualityMonitor.kicad_sch (KiCad schematic)
At the start: 15 parts, among them J1 USB_C_Receptacle_USB2.0_16P, SW1 RESET, SW2 BOOT, U1 USBLC6-2SC6, U2 AP7361C-33E, U3 ESP32-S3-WROOM-1

Commit message: Add I2C bus pull ups and SHT40 sensor
Connections:
- net +3V3: no longer C5.1, SW1.1
- net at R3.2, U3.3 (EN): now also C5.1, SW1.1
Changed lines of the file:
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@@
 	)
 	(junction
-		(at 217.17 69.85)
+		(at 232.41 77.47)
+		(diameter 0)
+		(color 0 0 0 0)
+	)
+	(junction
+		(at 217.17 80.01)
 		(diameter 0)
 		(color 0 0 0 0)
@@
 	(junction
 		(at 252.73 43.18)
-		(diameter 0)
-		(color 0 0 0 0)
-	)
-	(junction
-		(at 209.55 77.47)
 		(diameter 0)
 		(color 0 0 0 0)
@@
 	(wire
 		(pts
-			(xy 203.2 77.47) (xy 209.55 77.47)
-		)
-		(stroke
-			(width 0)
-			(type default)
-		)
-	)
-	(wire
-		(pts
 			(xy 209.55 43.18) (xy 209.55 53.34)
 		)
@@
 	(wire
 		(pts
-			(xy 209.55 77.47) (xy 209.55 74.93)
-		)
-		(stroke
-			(width 0)
-			(type default)
-		)
-	)
-	(wire
-		(pts
 			(xy 63.5 101.6) (xy 63.5 102.87)
 		)
@@
 	(wire
 		(pts
-			(xy 217.17 77.47) (xy 217.17 81.28)
+			(xy 217.17 77.47) (xy 217.17 80.01)
 		)
 		(stroke
@@
 	(wire
 		(pts
+			(xy 232.41 80.01) (xy 232.41 77.47)
+		)
+		(stroke
+			(width 0)
+			(type default)
+		)
+	)
+	(wire
+		(pts
 			(xy 83.82 106.68) (xy 83.82 107.95)
 		)
@@
 	(wire
 		(pts
-			(xy 209.55 77.47) (xy 217.17 77.47)
+			(xy 203.2 77.47) (xy 217.17 77.47)
 		)
 		(stroke
@@
 	(wire
 		(pts
-			(xy 209.55 74.93) (xy 217.17 74.93)
-		)
-		(stroke
-			(width 0)
-			(type default)
-		)
-	)
-	(wire
-		(pts
 			(xy 63.5 105.41) (xy 63.5 107.95)
 		)
@@
 	(wire
 		(pts
+			(xy 217.17 80.01) (xy 217.17 81.28)
+		)
+		(stroke
+			(width 0)
+			(type default)
+		)
+	)
+	(wire
+		(pts
 			(xy 269.24 87.63) (xy 270.51 87.63)
 		)
@@
 	(wire
 		(pts
+			(xy 217.17 80.01) (xy 232.41 80.01)
+		)
+		(stroke
+			(width 0)
+			(type default)
+		)
+	)
+	(wire
+		(pts
 			(xy 149.86 104.14) (xy 153.67 104.14)
 		)
 		(stroke
-			(width 0)
-			(type default)
-		)
-	)
-	(wire
-		(pts
-			(xy 217.17 69.85) (xy 217.17 74.93)
-		)
-		(stroke
